Commit message: fix: move lidar a bit downwards

File: src/omni_robot/urdf/omni_robot.urdf.xacro (robot description, xacro)
@@ -25,5 +25,5 @@
   </link>
   <!-- LiDAR (2D, 360°) mounted on top -->
-  <xacro:property name="lidar_z" value="${robot_height + 0.05}" />
+  <xacro:property name="lidar_z" value="${robot_height + 0.01}" />
   <joint name="lidar_joint" type="fixed">
     <parent link="base_link"/>
